File: RelayBoard.kicad_pcb (KiCad board)
At the start: 2 copper layers, 0 parts

Commit message: Started laying out PCB
Parts:
- added P1: HE10-32, Pin_Headers:Pin_Header_Straight_1x32, F.Cu at (-253.6, 81.8)
- added P2: CONN_2, Pin_Headers:Pin_Header_Straight_1x02, F.Cu at (-153.0, 142.7)
- added Q1: NPN, Discret:TO18CBE, F.Cu at (-177.2, 141.0)
- added Q10: NPN, Discret:TO18CBE, F.Cu at (-174.9, 132.5)
- added Q11: NPN, Discret:TO18CBE, F.Cu at (-152.0, 102.5)
- added Q12: NPN, Discret:TO18CBE, F.Cu at (-182.1, 132.5)
- added Q13: NPN, Discret:TO18CBE, F.Cu at (-129.4, 83.2)
- added Q14: NPN, Discret:TO18CBE, F.Cu at (-191.7, 138.2)
- added Q15: NPN, Discret:TO18CBE, F.Cu at (-122.2, 91.7)
- added Q16: NPN, Discret:TO18CBE, F.Cu at (-209.6, 173.8)
- added Q17: NPN, Discret:TO18CBE, F.Cu at (-184.4, 149.4)
- added Q18: NPN, Discret:TO18CBE, F.Cu at (-137.5, 99.6)
- added Q19: NPN, Discret:TO18CBE, F.Cu at (-167.7, 132.5)
- added Q2: NPN, Discret:TO18CBE, F.Cu at (-191.7, 155.2)
- added Q20: NPN, Discret:TO18CBE, F.Cu at (-144.8, 111.0)
- added Q21: NPN, Discret:TO18CBE, F.Cu at (-152.0, 119.4)
- added Q22: NPN, Discret:TO18CBE, F.Cu at (-202.4, 173.8)
- added Q23: NPN, Discret:TO18CBE, F.Cu at (-137.5, 108.1)
- added Q24: NPN, Discret:TO18CBE, F.Cu at (-224.1, 173.6)
- added Q25: NPN, Discret:TO18CBE, F.Cu at (-130.3, 100.1)
- added Q26: NPN, Discret:TO18CBE, F.Cu at (-170.0, 141.0)
- added Q27: NPN, Discret:TO18CBE, F.Cu at (-195.2, 165.3)
- added Q28: NPN, Discret:TO18CBE, F.Cu at (-177.2, 149.4)
- added Q29: NPN, Discret:TO18CBE, F.Cu at (-160.4, 132.5)
- added Q3: NPN, Discret:TO18CBE, F.Cu at (-202.4, 165.3)
- added Q30: NPN, Discret:TO18CBE, F.Cu at (-122.2, 83.2)
- added Q31: NPN, Discret:TO18CBE, F.Cu at (-129.4, 91.7)
- added Q32: NPN, Discret:TO18CBE, F.Cu at (-231.3, 173.6)
- added Q4: NPN, Discret:TO18CBE, F.Cu at (-209.6, 165.3)
- added Q5: NPN, Discret:TO18CBE, F.Cu at (-216.9, 170.7)
- added Q6: NPN, Discret:TO18CBE, F.Cu at (-191.7, 146.7)
- added Q7: NPN, Discret:TO18CBE, F.Cu at (-184.4, 141.0)
- added Q8: NPN, Discret:TO18CBE, F.Cu at (-152.0, 111.0)
- added Q9: NPN, Discret:TO18CBE, F.Cu at (-144.8, 102.5)
- added R1: 1K, Discret:R3, F.Cu at (-270.8, 169.9)
- added R10: 1K, Discret:R3, F.Cu at (-261.3, 175.7)
- added R11: 1K, Discret:R3, F.Cu at (-270.8, 175.7)
- added R12: 1K, Discret:R3, F.Cu at (-280.4, 175.7)
- added R13: 1K, Discret:R3, F.Cu at (-261.3, 172.8)
- added R14: 1K, Discret:R3, F.Cu at (-270.8, 172.8)
- added R15: 1K, Discret:R3, F.Cu at (-261.3, 169.9)
- added R16: 1K, Discret:R3, F.Cu at (-270.8, 167.0)
- added R17: 1K, Discret:R3, F.Cu at (-261.3, 167.0)
- added R18: 1K, Discret:R3, F.Cu at (-250.2, 84.9)
- added R19: 1K, Discret:R3, F.Cu at (-240.7, 84.9)
- added R2: 1K, Discret:R3, F.Cu at (-151.1, 95.9)
- added R20: 1K, Discret:R3, F.Cu at (-250.2, 87.8)
- added R21: 1K, Discret:R3, F.Cu at (-240.7, 87.8)
- added R22: 1K, Discret:R3, F.Cu at (-250.2, 90.6)
- added R23: 1K, Discret:R3, F.Cu at (-240.7, 90.6)
- added R24: 1K, Discret:R3, F.Cu at (-289.9, 167.0)
- added R25: 1K, Discret:R3, F.Cu at (-289.9, 169.9)
- added R26: 1K, Discret:R3, F.Cu at (-289.9, 172.8)
- added R27: 1K, Discret:R3, F.Cu at (-280.4, 167.0)
- added R28: 1K, Discret:R3, F.Cu at (-280.4, 169.9)
- added R29: 1K, Discret:R3, F.Cu at (-289.9, 175.7)
- added R3: 1K, Discret:R3, F.Cu at (-190.7, 128.8)
- added R30: 1K, Discret:R3, F.Cu at (-289.9, 178.5)
- added R31: 1K, Discret:R3, F.Cu at (-280.4, 172.8)
- added R32: 1K, Discret:R3, F.Cu at (-190.7, 131.7)
- added R4: 1K, Discret:R3, F.Cu at (-242.3, 178.1)
- added R5: 1K, Discret:R3, F.Cu at (-230.4, 167.0)
- added R6: 1K, Discret:R3, F.Cu at (-251.8, 178.1)
- added R7: 1K, Discret:R3, F.Cu at (-261.3, 178.5)
- added R8: 1K, Discret:R3, F.Cu at (-270.8, 178.5)
- added R9: 1K, Discret:R3, F.Cu at (-280.4, 178.5)
- added RE1: R-SPDT, RelayLib:R-SPDT, F.Cu at (37.5, 69.2)
- added RE10: R-SPDT, RelayLib:R-SPDT, F.Cu at (-294.1, 116.8)
- added RE11: R-SPDT, RelayLib:R-SPDT, F.Cu at (-274.3, 100.4)
- added RE12: R-SPDT, RelayLib:R-SPDT, F.Cu at (-254.5, 95.0)
- added RE13: R-SPDT, RelayLib:R-SPDT, F.Cu at (-294.1, 100.4)
- added RE14: R-SPDT, RelayLib:R-SPDT, F.Cu at (-274.3, 84.0)
- added RE15: R-SPDT, RelayLib:R-SPDT, F.Cu at (-294.1, 84.0)
- added RE16: R-SPDT, RelayLib:R-SPDT, F.Cu at (-214.8, 144.3)
- added RE17: R-SPDT, RelayLib:R-SPDT, F.Cu at (-211.5, 74.8)
- added RE18: R-SPDT, RelayLib:R-SPDT, F.Cu at (-171.8, 74.8)
- added RE19: R-SPDT, RelayLib:R-SPDT, F.Cu at (-254.5, 144.3)
- added RE2: R-SPDT, RelayLib:R-SPDT, F.Cu at (55.2, 69.2)
- added RE20: R-SPDT, RelayLib:R-SPDT, F.Cu at (-234.6, 116.8)
- added RE21: R-SPDT, RelayLib:R-SPDT, F.Cu at (-195.0, 95.0)
- added RE22: R-SPDT, RelayLib:R-SPDT, F.Cu at (-234.6, 133.3)
- added RE23: R-SPDT, RelayLib:R-SPDT, F.Cu at (-214.8, 111.5)
- added RE24: R-SPDT, RelayLib:R-SPDT, F.Cu at (-175.2, 95.0)
- added RE25: R-SPDT, RelayLib:R-SPDT, F.Cu at (-274.3, 149.7)
- added RE26: R-SPDT, RelayLib:R-SPDT, F.Cu at (-195.0, 111.5)
- added RE27: R-SPDT, RelayLib:R-SPDT, F.Cu at (-214.8, 127.9)
- added RE28: R-SPDT, RelayLib:R-SPDT, F.Cu at (-234.6, 149.7)
- added RE29: R-SPDT, RelayLib:R-SPDT, F.Cu at (-254.5, 160.8)
- added RE3: R-SPDT, RelayLib:R-SPDT, F.Cu at (73.0, 69.2)
- added RE30: R-SPDT, RelayLib:R-SPDT, F.Cu at (-152.0, 74.8)
- added RE31: R-SPDT, RelayLib:R-SPDT, F.Cu at (-175.2, 111.5)
- added RE32: R-SPDT, RelayLib:R-SPDT, F.Cu at (-254.5, 127.9)
- added RE4: R-SPDT, RelayLib:R-SPDT, F.Cu at (-294.1, 149.7)
- added RE5: R-SPDT, RelayLib:R-SPDT, F.Cu at (-274.3, 133.3)
- added RE6: R-SPDT, RelayLib:R-SPDT, F.Cu at (-234.6, 84.0)
- added RE7: R-SPDT, RelayLib:R-SPDT, F.Cu at (-294.1, 133.3)
- added RE8: R-SPDT, RelayLib:R-SPDT, F.Cu at (-274.3, 116.8)
- added RE9: R-SPDT, RelayLib:R-SPDT, F.Cu at (-191.6, 74.8)
- added TB1: TermBlk, Socket_Strips:Socket_Strip_Straight_1x03, F.Cu at (29.8, 66.0)
- added TB10: TermBlk, Socket_Strips:Socket_Strip_Straight_1x03, F.Cu at (-127.6, 114.9)
- added TB11: TermBlk, Socket_Strips:Socket_Strip_Straight_1x03, F.Cu at (-134.9, 120.6)
- added TB12: TermBlk, Socket_Strips:Socket_Strip_Straight_1x03, F.Cu at (-121.6, 109.6)
- added TB13: TermBlk, Socket_Strips:Socket_Strip_Straight_1x03, F.Cu at (-167.3, 153.5)
- added TB14: TermBlk, Socket_Strips:Socket_Strip_Straight_1x03, F.Cu at (-186.4, 172.7)
- added TB15: TermBlk, Socket_Strips:Socket_Strip_Straight_1x03, F.Cu at (-161.2, 145.0)
- added TB16: TermBlk, Socket_Strips:Socket_Strip_Straight_1x03, F.Cu at (-121.6, 104.2)
- added TB17: TermBlk, Socket_Strips:Socket_Strip_Straight_1x03, F.Cu at (-175.7, 161.9)
- added TB18: TermBlk, Socket_Strips:Socket_Strip_Straight_1x03, F.Cu at (-152.9, 137.3)
- added TB19: TermBlk, Socket_Strips:Socket_Strip_Straight_1x03, F.Cu at (-184.1, 156.6)
- added TB2: TermBlk, Socket_Strips:Socket_Strip_Straight_1x03, F.Cu at (-143.3, 128.9)
- added TB20: TermBlk, Socket_Strips:Socket_Strip_Straight_1x03, F.Cu at (-151.6, 126.6)
- added TB21: TermBlk, Socket_Strips:Socket_Strip_Straight_1x03, F.Cu at (-184.1, 161.9)
- added TB22: TermBlk, Socket_Strips:Socket_Strip_Straight_1x03, F.Cu at (-169.6, 148.1)
- added TB23: TermBlk, Socket_Strips:Socket_Strip_Straight_1x03, F.Cu at (-194.8, 172.5)
- added TB24: TermBlk, Socket_Strips:Socket_Strip_Straight_1x03, F.Cu at (-162.4, 139.6)
- added TB25: TermBlk, Socket_Strips:Socket_Strip_Straight_1x03, F.Cu at (-122.7, 98.8)
- added TB26: TermBlk, Socket_Strips:Socket_Strip_Straight_1x03, F.Cu at (-129.9, 107.3)
- added TB27: TermBlk, Socket_Strips:Socket_Strip_Straight_1x03, F.Cu at (-175.7, 156.6)
- added TB28: TermBlk, Socket_Strips:Socket_Strip_Straight_1x03, F.Cu at (-152.9, 132.0)
- added TB29: TermBlk, Socket_Strips:Socket_Strip_Straight_1x03, F.Cu at (-136.0, 115.2)
- added TB3: TermBlk, Socket_Strips:Socket_Strip_Straight_1x03, F.Cu at (-186.4, 178.1)
- added TB30: TermBlk, Socket_Strips:Socket_Strip_Straight_1x03, F.Cu at (-143.3, 123.5)
- added TB31: TermBlk, Socket_Strips:Socket_Strip_Straight_1x03, F.Cu at (-194.8, 177.8)
- added TB32: TermBlk, Socket_Strips:Socket_Strip_Straight_1x03, F.Cu at (-186.4, 167.3)
- added TB4: TermBlk, Socket_Strips:Socket_Strip_Straight_1x03, F.Cu at (-158.9, 150.4)
- added TB5: TermBlk, Socket_Strips:Socket_Strip_Straight_1x03, F.Cu at (-126.5, 120.3)
- added TB6: TermBlk, Socket_Strips:Socket_Strip_Straight_1x03, F.Cu at (-167.3, 158.8)
- added TB7: TermBlk, Socket_Strips:Socket_Strip_Straight_1x03, F.Cu at (-178.0, 167.3)
- added TB8: TermBlk, Socket_Strips:Socket_Strip_Straight_1x03, F.Cu at (-144.5, 134.2)
- added TB9: TermBlk, Socket_Strips:Socket_Strip_Straight_1x03, F.Cu at (-134.9, 126.0)

Commit message: Update
* Updated Readme with a warning.
* The schematic is nowhere near done as I forgot to include diodes to
  protect against the feedback from relays turning on and off.
Parts:
- moved RE7 442.9 mm to (144.1, 69.2), turned to 270 degrees
- moved RE8 438.2 mm to (161.3, 69.2), turned to 270 degrees
- moved RE4 393.3 mm to (90.8, 69.2), turned to 270 degrees
- moved RE5 388.2 mm to (108.6, 69.2), turned to 270 degrees
- moved P1 368.6 mm to (114.3, 103.5)
- moved RE6 361.3 mm to (126.4, 69.2), turned to 270 degrees
Changed lines of the file:
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@@
     (links 256)
     (no_connects 256)
-    (area 0 0 0 0)
+    (area -294.64 64.388999 161.794 179.9852)
     (thickness 1.6)
     (drawings 0)
@@
     (pad_to_mask_clearance 0)
     (aux_axis_origin 0 0)
-    (visible_elements FFFFFF7F)
+    (visible_elements FFFFF77F)
     (pcbplotparams
       (layerselection 3178497)
@@
   )
   (module Pin_Headers:Pin_Header_Straight_1x32 (layer F.Cu)
-    (at -253.618999 81.8388)
+    (at 114.3 103.505)
     (descr "1 pin")
     (tags "CONN DEV")
@@
   )
   (module RelayLib:R-SPDT (layer F.Cu)
-    (at -294.136 149.709)
-    (fp_text reference RE4 (at 12 5.8) (layer F.SilkS)
+    (at 90.805 69.215 270)
+    (fp_text reference RE4 (at 12 5.8 270) (layer F.SilkS)
       (effects (font (size 1.5 1.5) (thickness 0.15)))
     )
-    (fp_text value R-SPDT (at 9.8 9.2) (layer F.SilkS)
+    (fp_text value R-SPDT (at 9.8 9.2 270) (layer F.SilkS)
       (effects (font (size 1.5 1.5) (thickness 0.15)))
     )
@@
     (fp_line (start 19 15.6) (end 19 0) (layer F.SilkS) (width 0.15))
     (fp_line (start 19 0) (end 0 0) (layer F.SilkS) (width 0.15))
-    (pad 5 thru_hole circle (at 3.4 1.8) (size 1.524 1.524) (drill 1.3) (layers *.Cu *.Mask F.SilkS)
+    (pad 5 thru_hole circle (at 3.4 1.8 270) (size 1.524 1.524) (drill 1.3) (layers *.Cu *.Mask F.SilkS)
       (net 33 +5V))
-    (pad 4 thru_hole circle (at 3.4 13.8) (size 1.524 1.524) (drill 1.3) (layers *.Cu *.Mask F.SilkS)
+    (pad 4 thru_hole circle (at 3.4 13.8 270) (size 1.524 1.524) (drill 1.3) (layers *.Cu *.Mask F.SilkS)
       (net 42 "Net-(Q4-Pad3)"))
-    (pad 2 thru_hole circle (at 1.4 7.8) (size 1.524 1.524) (drill 1.3) (layers *.Cu *.Mask F.SilkS)
+    (pad 2 thru_hole circle (at 1.4 7.8 270) (size 1.524 1.524) (drill 1.3) (layers *.Cu *.Mask F.SilkS)
       (net 108 "Net-(RE4-Pad2)"))
-    (pad 1 thru_hole circle (at 15.6 1.8) (size 1.524 1.524) (drill 1.3) (layers *.Cu *.Mask F.SilkS)
+    (pad 1 thru_hole circle (at 15.6 1.8 270) (size 1.524 1.524) (drill 1.3) (layers *.Cu *.Mask F.SilkS)
       (net 109 "Net-(RE4-Pad1)"))
-    (pad 3 thru_hole circle (at 15.6 13.8) (size 1.524 1.524) (drill 1.3) (layers *.Cu *.Mask F.SilkS)
+    (pad 3 thru_hole circle (at 15.6 13.8 270) (size 1.524 1.524) (drill 1.3) (layers *.Cu *.Mask F.SilkS)
       (net 110 "Net-(RE4-Pad3)"))
   )
   (module RelayLib:R-SPDT (layer F.Cu)
-    (at -274.306 133.279)
-    (fp_text reference RE5 (at 12 5.8) (layer F.SilkS)
+    (at 108.585 69.215 270)
+    (fp_text reference RE5 (at 9.511 5.786 270) (layer F.SilkS)
       (effects (font (size 1.5 1.5) (thickness 0.15)))
     )
-    (fp_text value R-SPDT (at 9.8 9.2) (layer F.SilkS)
+    (fp_text value R-SPDT (at 9.8 9.2 270) (layer F.SilkS)
       (effects (font (size 1.5 1.5) (thickness 0.15)))
     )
@@
     (fp_line (start 19 15.6) (end 19 0) (layer F.SilkS) (width 0.15))
     (fp_line (start 19 0) (end 0 0) (layer F.SilkS) (width 0.15))
-    (pad 5 thru_hole circle (at 3.4 1.8) (size 1.524 1.524) (drill 1.3) (layers *.Cu *.Mask F.SilkS)
+    (pad 5 thru_hole circle (at 3.4 1.8 270) (size 1.524 1.524) (drill 1.3) (layers *.Cu *.Mask F.SilkS)
       (net 33 +5V))
-    (pad 4 thru_hole circle (at 3.4 13.8) (size 1.524 1.524) (drill 1.3) (layers *.Cu *.Mask F.SilkS)
+    (pad 4 thru_hole circle (at 3.4 13.8 270) (size 1.524 1.524) (drill 1.3) (layers *.Cu *.Mask F.SilkS)
       (net 44 "Net-(Q5-Pad3)"))
-    (pad 2 thru_hole circle (at 1.4 7.8) (size 1.524 1.524) (drill 1.3) (layers *.Cu *.Mask F.SilkS)
+    (pad 2 thru_hole circle (at 1.4 7.8 270) (size 1.524 1.524) (drill 1.3) (layers *.Cu *.Mask F.SilkS)
       (net 111 "Net-(RE5-Pad2)"))
-    (pad 1 thru_hole circle (at 15.6 1.8) (size 1.524 1.524) (drill 1.3) (layers *.Cu *.Mask F.SilkS)
+    (pad 1 thru_hole circle (at 15.6 1.8 270) (size 1.524 1.524) (drill 1.3) (layers *.Cu *.Mask F.SilkS)
       (net 112 "Net-(RE5-Pad1)"))
-    (pad 3 thru_hole circle (at 15.6 13.8) (size 1.524 1.524) (drill 1.3) (layers *.Cu *.Mask F.SilkS)
+    (pad 3 thru_hole circle (at 15.6 13.8 270) (size 1.524 1.524) (drill 1.3) (layers *.Cu *.Mask F.SilkS)
       (net 113 "Net-(RE5-Pad3)"))
   )
   (module RelayLib:R-SPDT (layer F.Cu)
-    (at -234.646 83.989)
-    (fp_text reference RE6 (at 12 5.8) (layer F.SilkS)
+    (at 126.365 69.215 270)
+    (fp_text reference RE6 (at 12 5.8 270) (layer F.SilkS)
       (effects (font (size 1.5 1.5) (thickness 0.15)))
     )
-    (fp_text value R-SPDT (at 9.8 9.2) (layer F.SilkS)
+    (fp_text value R-SPDT (at 9.8 9.2 270) (layer F.SilkS)
       (effects (font (size 1.5 1.5) (thickness 0.15)))
     )
@@
     (fp_line (start 19 15.6) (end 19 0) (layer F.SilkS) (width 0.15))
     (fp_line (start 19 0) (end 0 0) (layer F.SilkS) (width 0.15))
-    (pad 5 thru_hole circle (at 3.4 1.8) (size 1.524 1.524) (drill 1.3) (layers *.Cu *.Mask F.SilkS)
+    (pad 5 thru_hole circle (at 3.4 1.8 270) (size 1.524 1.524) (drill 1.3) (layers *.Cu *.Mask F.SilkS)
       (net 33 +5V))
-    (pad 4 thru_hole circle (at 3.4 13.8) (size 1.524 1.524) (drill 1.3) (layers *.Cu *.Mask F.SilkS)
+    (pad 4 thru_hole circle (at 3.4 13.8 270) (size 1.524 1.524) (drill 1.3) (layers *.Cu *.Mask F.SilkS)
       (net 46 "Net-(Q6-Pad3)"))
-    (pad 2 thru_hole circle (at 1.4 7.8) (size 1.524 1.524) (drill 1.3) (layers *.Cu *.Mask F.SilkS)
+    (pad 2 thru_hole circle (at 1.4 7.8 270) (size 1.524 1.524) (drill 1.3) (layers *.Cu *.Mask F.SilkS)
       (net 114 "Net-(RE6-Pad2)"))
-    (pad 1 thru_hole circle (at 15.6 1.8) (size 1.524 1.524) (drill 1.3) (layers *.Cu *.Mask F.SilkS)
+    (pad 1 thru_hole circle (at 15.6 1.8 270) (size 1.524 1.524) (drill 1.3) (layers *.Cu *.Mask F.SilkS)
       (net 115 "Net-(RE6-Pad1)"))
-    (pad 3 thru_hole circle (at 15.6 13.8) (size 1.524 1.524) (drill 1.3) (layers *.Cu *.Mask F.SilkS)
+    (pad 3 thru_hole circle (at 15.6 13.8 270) (size 1.524 1.524) (drill 1.3) (layers *.Cu *.Mask F.SilkS)
       (net 116 "Net-(RE6-Pad3)"))
   )
   (module RelayLib:R-SPDT (layer F.Cu)
-    (at -294.136 133.279)
-    (fp_text reference RE7 (at 12 5.8) (layer F.SilkS)
+    (at 144.145 69.215 270)
+    (fp_text reference RE7 (at 12 5.8 270) (layer F.SilkS)
       (effects (font (size 1.5 1.5) (thickness 0.15)))
     )
-    (fp_text value R-SPDT (at 9.8 9.2) (layer F.SilkS)
+    (fp_text value R-SPDT (at 9.8 9.2 270) (layer F.SilkS)
       (effects (font (size 1.5 1.5) (thickness 0.15)))
     )
@@
     (fp_line (start 19 15.6) (end 19 0) (layer F.SilkS) (width 0.15))
     (fp_line (start 19 0) (end 0 0) (layer F.SilkS) (width 0.15))
-    (pad 5 thru_hole circle (at 3.4 1.8) (size 1.524 1.524) (drill 1.3) (layers *.Cu *.Mask F.SilkS)
+    (pad 5 thru_hole circle (at 3.4 1.8 270) (size 1.524 1.524) (drill 1.3) (layers *.Cu *.Mask F.SilkS)
       (net 33 +5V))
-    (pad 4 thru_hole circle (at 3.4 13.8) (size 1.524 1.524) (drill 1.3) (layers *.Cu *.Mask F.SilkS)
+    (pad 4 thru_hole circle (at 3.4 13.8 270) (size 1.524 1.524) (drill 1.3) (layers *.Cu *.Mask F.SilkS)
       (net 48 "Net-(Q7-Pad3)"))
-    (pad 2 thru_hole circle (at 1.4 7.8) (size 1.524 1.524) (drill 1.3) (layers *.Cu *.Mask F.SilkS)
+    (pad 2 thru_hole circle (at 1.4 7.8 270) (size 1.524 1.524) (drill 1.3) (layers *.Cu *.Mask F.SilkS)
       (net 117 "Net-(RE7-Pad2)"))
-    (pad 1 thru_hole circle (at 15.6 1.8) (size 1.524 1.524) (drill 1.3) (layers *.Cu *.Mask F.SilkS)
+    (pad 1 thru_hole circle (at 15.6 1.8 270) (size 1.524 1.524) (drill 1.3) (layers *.Cu *.Mask F.SilkS)
       (net 118 "Net-(RE7-Pad1)"))
-    (pad 3 thru_hole circle (at 15.6 13.8) (size 1.524 1.524) (drill 1.3) (layers *.Cu *.Mask F.SilkS)
+    (pad 3 thru_hole circle (at 15.6 13.8 270) (size 1.524 1.524) (drill 1.3) (layers *.Cu *.Mask F.SilkS)
       (net 119 "Net-(RE7-Pad3)"))
   )
   (module RelayLib:R-SPDT (layer F.Cu)
-    (at -274.306 116.849)
-    (fp_text reference RE8 (at 12 5.8) (layer F.SilkS)
+    (at 161.29 69.215 270)
+    (fp_text reference RE8 (at 12 5.8 270) (layer F.SilkS)
       (effects (font (size 1.5 1.5) (thickness 0.15)))
     )
-    (fp_text value R-SPDT (at 9.8 9.2) (layer F.SilkS)
+    (fp_text value R-SPDT (at 9.8 9.2 270) (layer F.SilkS)
       (effects (font (size 1.5 1.5) (thickness 0.15)))
     )
@@
     (fp_line (start 19 15.6) (end 19 0) (layer F.SilkS) (width 0.15))
     (fp_line (start 19 0) (end 0 0) (layer F.SilkS) (width 0.15))
-    (pad 5 thru_hole circle (at 3.4 1.8) (size 1.524 1.524) (drill 1.3) (layers *.Cu *.Mask F.SilkS)
+    (pad 5 thru_hole circle (at 3.4 1.8 270) (size 1.524 1.524) (drill 1.3) (layers *.Cu *.Mask F.SilkS)
       (net 33 +5V))
-    (pad 4 thru_hole circle (at 3.4 13.8) (size 1.524 1.524) (drill 1.3) (layers *.Cu *.Mask F.SilkS)
+    (pad 4 thru_hole circle (at 3.4 13.8 270) (size 1.524 1.524) (drill 1.3) (layers *.Cu *.Mask F.SilkS)
       (net 50 "Net-(Q8-Pad3)"))
-    (pad 2 thru_hole circle (at 1.4 7.8) (size 1.524 1.524) (drill 1.3) (layers *.Cu *.Mask F.SilkS)
+    (pad 2 thru_hole circle (at 1.4 7.8 270) (size 1.524 1.524) (drill 1.3) (layers *.Cu *.Mask F.SilkS)
       (net 120 "Net-(RE8-Pad2)"))
-    (pad 1 thru_hole circle (at 15.6 1.8) (size 1.524 1.524) (drill 1.3) (layers *.Cu *.Mask F.SilkS)
+    (pad 1 thru_hole circle (at 15.6 1.8 270) (size 1.524 1.524) (drill 1.3) (layers *.Cu *.Mask F.SilkS)
       (net 121 "Net-(RE8-Pad1)"))
-    (pad 3 thru_hole circle (at 15.6 13.8) (size 1.524 1.524) (drill 1.3) (layers *.Cu *.Mask F.SilkS)
+    (pad 3 thru_hole circle (at 15.6 13.8 270) (size 1.524 1.524) (drill 1.3) (layers *.Cu *.Mask F.SilkS)
       (net 122 "Net-(RE8-Pad3)"))
   )

Commit message: Placed Most of the relays on the PCB
Parts:
- added D1: DIODE, Discret:D3, F.Cu at (41.9, 73.7)
- added D10: DIODE, Discret:D3, F.Cu at (-89.3, 138.1)
- added D11: DIODE, Discret:D3, F.Cu at (-161.8, 212.0)
- added D12: DIODE, Discret:D3, F.Cu at (-161.8, 209.2)
- added D13: DIODE, Discret:D3, F.Cu at (-152.3, 214.9)
- added D14: DIODE, Discret:D3, F.Cu at (-53.8, 121.1)
- added D15: DIODE, Discret:D3, F.Cu at (-63.3, 129.6)
- added D16: DIODE, Discret:D3, F.Cu at (-89.3, 155.2)
- added D17: DIODE, Discret:D3, F.Cu at (-73.6, 134.7)
- added D18: DIODE, Discret:D3, F.Cu at (-63.3, 126.8)
- added D19: DIODE, Discret:D3, F.Cu at (-63.3, 123.9)
- added D2: DIODE, Discret:D3, F.Cu at (-172.1, 129.3)
- added D20: DIODE, Discret:D3, F.Cu at (-63.3, 121.1)
- added D21: DIODE, Discret:D3, F.Cu at (-79.8, 143.2)
- added D22: DIODE, Discret:D3, F.Cu at (-53.8, 118.3)
- added D23: DIODE, Discret:D3, F.Cu at (-89.3, 152.3)
- added D24: DIODE, Discret:D3, F.Cu at (-79.8, 140.4)
- added D25: DIODE, Discret:D3, F.Cu at (-79.8, 137.6)
- added D26: DIODE, Discret:D3, F.Cu at (-162.6, 220.6)
- added D27: DIODE, Discret:D3, F.Cu at (-162.6, 217.7)
- added D28: DIODE, Discret:D3, F.Cu at (-89.3, 143.8)
- added D29: DIODE, Discret:D3, F.Cu at (-89.3, 146.6)
- added D3: DIODE, Discret:D3, F.Cu at (-221.3, 212.1)
- added D30: DIODE, Discret:D3, F.Cu at (-116.0, 174.4)
- added D31: DIODE, Discret:D3, F.Cu at (-89.3, 149.5)
- added D32: DIODE, Discret:D3, F.Cu at (-181.6, 126.5)
- added D4: DIODE, Discret:D3, F.Cu at (-181.6, 129.3)
- added D5: DIODE, Discret:D3, F.Cu at (108.0, 74.3)
- added D6: DIODE, Discret:D3, F.Cu at (-172.1, 123.6)
- added D7: DIODE, Discret:D3, F.Cu at (-181.6, 123.6)
- added D8: DIODE, Discret:D3, F.Cu at (-181.6, 219.7)
- added D9: DIODE, Discret:D3, F.Cu at (-63.3, 118.3)
- moved RE19 461.9 mm to (198.1, 52.1), turned to 270 degrees
- moved RE15 460.3 mm to (165.1, 52.1), turned to 270 degrees
- moved RE23 449.9 mm to (231.1, 52.1), turned to 270 degrees
- moved RE13 445.4 mm to (148.6, 52.1), turned to 270 degrees
- moved RE22 435.3 mm to (200.7, 133.3), turned to 90 degrees
- moved RE20 419.1 mm to (184.2, 133.3), turned to 90 degrees
- moved RE14 411.9 mm to (134.6, 133.3), turned to 90 degrees
- moved RE21 411.9 mm to (214.6, 52.1), turned to 270 degrees
- moved RE11 409.3 mm to (132.1, 52.1), turned to 270 degrees
- moved RE10 396.1 mm to (101.6, 133.3), turned to 90 degrees
- moved RE24 394.2 mm to (217.2, 133.3), turned to 90 degrees
- moved RE17 393.7 mm to (181.6, 52.1), turned to 270 degrees
- moved R1 381.4 mm to (101.6, 87.6), turned to 270 degrees
- moved RE12 374.6 mm to (118.1, 133.3), turned to 90 degrees
- moved RE16 366.1 mm to (151.1, 133.3), turned to 90 degrees
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
Commit message: Placed all of the relays on the PCB.
Parts:
- moved RE31 507.8 mm to (297.2, 52.1), turned to 270 degrees
- moved RE25 493.4 mm to (247.7, 52.1), turned to 270 degrees
- moved RE29 480.4 mm to (280.7, 52.1), turned to 270 degrees
- moved RE30 475.6 mm to (266.7, 133.3), turned to 90 degrees
- moved RE26 459.3 mm to (233.7, 133.3), turned to 90 degrees
- moved RE32 427.0 mm to (283.2, 133.3), turned to 90 degrees
- moved RE27 418.5 mm to (264.2, 52.1), turned to 270 degrees
- moved RE28 416.3 mm to (250.2, 133.3), turned to 90 degrees

Commit message: Placed all of the terminal blocks on the PCB.
Parts:
- moved TB29 416.3 mm to (273.1, 48.3), turned to 180 degrees
- moved TB28 386.4 mm to (257.8, 146.1)
- moved TB27 379.1 mm to (256.5, 48.3), turned to 180 degrees
- moved TB19 377.2 mm to (190.5, 48.3), turned to 180 degrees
- moved TB32 365.9 mm to (290.8, 146.1)
- moved TB20 353.3 mm to (191.8, 146.1)
- moved TB31 353.1 mm to (289.6, 48.3), turned to 180 degrees
- moved TB30 349.9 mm to (274.3, 146.1)
- moved TB26 347.7 mm to (241.3, 146.1)
- moved TB23 328.7 mm to (223.5, 48.3), turned to 180 degrees
- moved TB25 307.8 mm to (240.0, 48.3), turned to 180 degrees
- moved TB21 301.3 mm to (207.0, 48.3), turned to 180 degrees
- moved TB24 291.7 mm to (224.8, 146.1)
- moved TB16 284.2 mm to (158.8, 146.1)
- moved TB15 278.5 mm to (157.5, 48.3), turned to 180 degrees
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Other:
- net class Default: trace_width 0.254 -> 0.95

Commit message: Did a bunch to the PCB Layout
* Diode Placement
* Tracks
* Commenting
Parts:
- moved D30 391.2 mm to (274.3, 148.6), turned to 180 degrees
- moved Q24 346.5 mm to (229.9, 119.4), turned to 180 degrees
- moved D13 336.7 mm to (141.0, 49.5)
- moved Q19 336.3 mm to (194.3, 78.7)
- moved D3 323.5 mm to (58.4, 49.5)
- moved Q25 314.8 mm to (243.8, 78.7)
- moved D6 249.6 mm to (76.2, 148.6), turned to 180 degrees
- moved R11 246.3 mm to (114.3, 100.3), turned to 90 degrees
- moved D15 234.9 mm to (157.5, 49.5)
- moved D2 216.2 mm to (43.2, 148.6), turned to 180 degrees
- moved Q8 212.0 mm to (95.2, 119.4), turned to 180 degrees
- moved Q12 211.2 mm to (128.3, 119.4), turned to 180 degrees
- moved Q16 206.5 mm to (161.3, 118.1), turned to 180 degrees
- moved Q13 205.4 mm to (144.8, 78.7)
- moved Q6 205.2 mm to (80.0, 119.4), turned to 180 degrees
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Routing:
- net +5V: track 0.00 -> 360.3 mm
- net Net-(RE6-Pad1): track 0.00 -> 30.0 mm
- net Net-(RE6-Pad3): track 0.00 -> 26.3 mm
- net Net-(RE6-Pad2): track 0.00 -> 7.82 mm
- net Net-(D6-Pad1): track 0.00 -> 7.06 mm
Other:
- board text added: "Board is 217mm x 118mm"

Commit message: Changed The Pin headers
* Changed Pin Headers
* Placed Most of the resistors on the board
Parts:
- P1: footprint Pin_Headers:Pin_Header_Straight_1x32 -> Pin_Headers:Pin_Header_Straight_2x16
- moved R27 515.1 mm to (285.8, 78.7), turned to 270 degrees
- moved R28 507.8 mm to (288.3, 120.7), turned to 90 degrees
- moved D32 506.0 mm to (323.9, 148.6), turned to 180 degrees
- moved D27 482.4 mm to (289.6, 49.5)
- moved R31 474.9 mm to (320.0, 77.5), turned to 270 degrees
- moved R32 467.2 mm to (320.0, 120.7), turned to 90 degrees
- moved D26 442.8 mm to (274.3, 148.6), turned to 180 degrees
- moved R25 441.2 mm to (269.2, 78.7), turned to 270 degrees
- moved Q30 440.9 mm to (311.1, 120.7), turned to 180 degrees
- moved R26 434.1 mm to (271.8, 119.4), turned to 90 degrees
- moved Q28 431.3 mm to (295.9, 120.7), turned to 180 degrees
- moved Q32 425.0 mm to (327.7, 120.7), turned to 180 degrees
- moved D31 423.8 mm to (322.6, 49.5)
- moved R23 414.6 mm to (254.0, 78.7), turned to 270 degrees
- moved Q31 408.9 mm to (327.7, 78.7)
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Routing:
- net +5V: track 360.3 -> 0.00 mm
- net Net-(RE2-Pad1): track 0.00 -> 28.9 mm
- net Net-(RE2-Pad3): track 0.00 -> 27.0 mm
- net Net-(RE2-Pad2): track 0.00 -> 7.82 mm
