File: RelayBoard.kicad_pcb (KiCad board)
At the start: 2 copper layers, 162 parts, among them P1 HE10-32, P2 CONN_2, Q1 NPN, Q10 NPN, Q11 NPN, Q12 NPN, Q13 NPN, Q14 NPN, Q15 NPN, Q16 NPN, Q17 NPN, Q18 NPN, Q19 NPN, Q2 NPN, Q20 NPN, Q21 NPN, Q22 NPN, Q23 NPN, Q24 NPN, Q25 NPN, Q26 NPN, Q27 NPN, Q28 NPN, Q29 NPN, Q3 NPN, Q30 NPN, Q31 NPN, Q32 NPN, Q4 NPN, Q5 NPN, Q6 NPN, Q7 NPN, Q8 NPN, Q9 NPN

Commit message: Finished Placing all parts on PCB
It's time to route the board
Parts:
- moved R29 488.7 mm to (303.5, 78.7), turned to 270 degrees
- moved R30 436.7 mm to (304.8, 120.7), turned to 90 degrees
- moved R18 326.1 mm to (204.5, 120.7), turned to 90 degrees
- moved R7 312.3 mm to (121.9, 77.5), turned to 270 degrees
- moved R10 45.5 mm to (138.4, 120.7)
Routing:
- net Net-(RE6-Pad1): track 30.0 -> 0.00 mm
- net Net-(RE2-Pad1): track 28.9 -> 0.00 mm
- net Net-(RE2-Pad3): track 27.0 -> 0.00 mm
- net Net-(RE6-Pad3): track 26.3 -> 0.00 mm
- net Net-(RE6-Pad2): track 7.82 -> 0.00 mm
- net Net-(RE2-Pad2): track 7.82 -> 0.00 mm
- net Net-(D6-Pad1): track 7.06 -> 0.00 mm
Changed lines of the file:
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@@
   (general
     (links 320)
-    (no_connects 313)
-    (area -184.15 19.05 344.17 180.34)
+    (no_connects 320)
+    (area 30.48 19.05 344.17 180.34)
     (thickness 1.6)
     (drawings 3)
-    (tracks 37)
+    (tracks 0)
     (zones 0)
     (modules 162)
@@
     (pad_to_mask_clearance 0)
     (aux_axis_origin 0 0)
-    (visible_elements FFFFF77F)
+    (visible_elements FFFFFF7F)
     (pcbplotparams
       (layerselection 3178497)
@@
   )
   (module Discret:R3 (layer F.Cu)
-    (at -179.3875 159.6697)
+    (at 121.92 77.47 270)
     (descr "Resitance 3 pas")
     (tags R)
     (autoplace_cost180 10)
-    (fp_text reference R7 (at 0 0.127) (layer F.SilkS) hide
+    (fp_text reference R7 (at 0 0.127 270) (layer F.SilkS) hide
       (effects (font (size 1.397 1.27) (thickness 0.2032)))
     )
-    (fp_text value 1K (at 0 0.127) (layer F.SilkS)
+    (fp_text value 1K (at 0 0.127 270) (layer F.SilkS)
       (effects (font (size 1.397 1.27) (thickness 0.2032)))
     )
@@
     (fp_line (start 3.302 1.016) (end 3.302 0) (layer F.SilkS) (width 0.2032))
     (fp_line (start -3.302 -0.508) (end -2.794 -1.016) (layer F.SilkS) (width 0.2032))
-    (pad 1 thru_hole circle (at -3.81 0) (size 1.397 1.397) (drill 0.8128) (layers *.Cu *.Mask F.SilkS)
+    (pad 1 thru_hole circle (at -3.81 0 270) (size 1.397 1.397) (drill 0.8128) (layers *.Cu *.Mask F.SilkS)
       (net 41 "Net-(Q7-Pad2)"))
-    (pad 2 thru_hole circle (at 3.81 0) (size 1.397 1.397) (drill 0.8128) (layers *.Cu *.Mask F.SilkS)
+    (pad 2 thru_hole circle (at 3.81 0 270) (size 1.397 1.397) (drill 0.8128) (layers *.Cu *.Mask F.SilkS)
       (net 20 Pin20))
     (model discret/resistor.wrl
@@
   )
   (module Discret:R3 (layer F.Cu)
-    (at 120.65 78.74 90)
+    (at 138.43 120.65 90)
     (descr "Resitance 3 pas")
     (tags R)
@@
   )
   (module Discret:R3 (layer F.Cu)
-    (at -119.8975 153.8997)
+    (at 204.47 120.65 90)
     (descr "Resitance 3 pas")
     (tags R)
     (autoplace_cost180 10)
-    (fp_text reference R18 (at 0 0.127) (layer F.SilkS) hide
+    (fp_text reference R18 (at 0 0.127 90) (layer F.SilkS) hide
       (effects (font (size 1.397 1.27) (thickness 0.2032)))
     )
-    (fp_text value 1K (at 0 0.127) (layer F.SilkS)
+    (fp_text value 1K (at 0 0.127 90) (layer F.SilkS)
       (effects (font (size 1.397 1.27) (thickness 0.2032)))
     )
@@
     (fp_line (start 3.302 1.016) (end 3.302 0) (layer F.SilkS) (width 0.2032))
     (fp_line (start -3.302 -0.508) (end -2.794 -1.016) (layer F.SilkS) (width 0.2032))
-    (pad 1 thru_hole circle (at -3.81 0) (size 1.397 1.397) (drill 0.8128) (layers *.Cu *.Mask F.SilkS)
+    (pad 1 thru_hole circle (at -3.81 0 90) (size 1.397 1.397) (drill 0.8128) (layers *.Cu *.Mask F.SilkS)
       (net 52 "Net-(Q18-Pad2)"))
-    (pad 2 thru_hole circle (at 3.81 0) (size 1.397 1.397) (drill 0.8128) (layers *.Cu *.Mask F.SilkS)
+    (pad 2 thru_hole circle (at 3.81 0 90) (size 1.397 1.397) (drill 0.8128) (layers *.Cu *.Mask F.SilkS)
       (net 9 Pin9))
     (model discret/resistor.wrl
@@
   )
   (module Discret:R3 (layer F.Cu)
-    (at -179.3875 153.9297)
+    (at 303.53 78.74 270)
     (descr "Resitance 3 pas")
     (tags R)
     (autoplace_cost180 10)
-    (fp_text reference R29 (at 0 0.127) (layer F.SilkS) hide
+    (fp_text reference R29 (at 0 0.127 270) (layer F.SilkS) hide
       (effects (font (size 1.397 1.27) (thickness 0.2032)))
     )
-    (fp_text value 1K (at 0 0.127) (layer F.SilkS)
+    (fp_text value 1K (at 0 0.127 270) (layer F.SilkS)
       (effects (font (size 1.397 1.27) (thickness 0.2032)))
     )
@@
     (fp_line (start 3.302 1.016) (end 3.302 0) (layer F.SilkS) (width 0.2032))
     (fp_line (start -3.302 -0.508) (end -2.794 -1.016) (layer F.SilkS) (width 0.2032))
-    (pad 1 thru_hole circle (at -3.81 0) (size 1.397 1.397) (drill 0.8128) (layers *.Cu *.Mask F.SilkS)
+    (pad 1 thru_hole circle (at -3.81 0 270) (size 1.397 1.397) (drill 0.8128) (layers *.Cu *.Mask F.SilkS)
       (net 63 "Net-(Q29-Pad2)"))
-    (pad 2 thru_hole circle (at 3.81 0) (size 1.397 1.397) (drill 0.8128) (layers *.Cu *.Mask F.SilkS)
+    (pad 2 thru_hole circle (at 3.81 0 270) (size 1.397 1.397) (drill 0.8128) (layers *.Cu *.Mask F.SilkS)
       (net 31 Pin31))
     (model discret/resistor.wrl
@@
   )
   (module Discret:R3 (layer F.Cu)
-    (at -130.2075 158.7397)
+    (at 304.8 120.65 90)
     (descr "Resitance 3 pas")
     (tags R)
     (autoplace_cost180 10)
-    (fp_text reference R30 (at 0 0.127) (layer F.SilkS) hide
+    (fp_text reference R30 (at 0 0.127 90) (layer F.SilkS) hide
       (effects (font (size 1.397 1.27) (thickness 0.2032)))
     )
-    (fp_text value 1K (at 0 0.127) (layer F.SilkS)
+    (fp_text value 1K (at 0 0.127 90) (layer F.SilkS)
       (effects (font (size 1.397 1.27) (thickness 0.2032)))
     )
@@
     (fp_line (start 3.302 1.016) (end 3.302 0) (layer F.SilkS) (width 0.2032))
     (fp_line (start -3.302 -0.508) (end -2.794 -1.016) (layer F.SilkS) (width 0.2032))
-    (pad 1 thru_hole circle (at -3.81 0) (size 1.397 1.397) (drill 0.8128) (layers *.Cu *.Mask F.SilkS)
+    (pad 1 thru_hole circle (at -3.81 0 90) (size 1.397 1.397) (drill 0.8128) (layers *.Cu *.Mask F.SilkS)
       (net 64 "Net-(Q30-Pad2)"))
-    (pad 2 thru_hole circle (at 3.81 0) (size 1.397 1.397) (drill 0.8128) (layers *.Cu *.Mask F.SilkS)
+    (pad 2 thru_hole circle (at 3.81 0 90) (size 1.397 1.397) (drill 0.8128) (layers *.Cu *.Mask F.SilkS)
       (net 15 Pin15))
     (model discret/resistor.wrl
@@
     (arrow2b (pts (xy 335.28 156.21) (xy 334.693579 155.083496)))
   )
-  (segment (start 76.2 144.83) (end 76.38 144.65) (width 0.95) (layer B.Cu) (net 70))
-  (segment (start 76.2 152.4) (end 76.2 144.83) (width 0.95) (layer B.Cu) (net 70))
-  (segment (start 72.03 130.45) (end 73.66 132.08) (width 0.95) (layer F.Cu) (net 71))
-  (segment (start 73.66 132.08) (end 73.66 143.51) (width 0.95) (layer F.Cu) (net 71))
-  (segment (start 73.66 143.51) (end 71.12 146.05) (width 0.95) (layer F.Cu) (net 71))
-  (segment (start 71.12 146.05) (end 69.85 146.05) (width 0.95) (layer F.Cu) (net 71))
-  (segment (start 69.85 146.05) (end 69.85 148.59) (width 0.95) (layer F.Cu) (net 71))
-  (segment (start 69.85 148.59) (end 69.85 149.86) (width 0.95) (layer F.Cu) (net 71))
-  (segment (start 69.85 149.86) (end 72.39 152.4) (width 0.95) (layer F.Cu) (net 71))
-  (segment (start 72.39 152.4) (end 73.66 152.4) (width 0.95) (layer F.Cu) (net 71))
-  (segment (start 70.38 130.45) (end 72.03 130.45) (width 0.95) (layer F.Cu) (net 71))
-  (segment (start 80.01 132.82) (end 82.38 130.45) (width 0.95) (layer F.Cu) (net 72))
-  (segment (start 80.01 144.78) (end 80.01 132.82) (width 0.95) (layer F.Cu) (net 72))
-  (segment (start 81.28 146.05) (end 80.01 144.78) (width 0.95) (layer F.Cu) (net 72))
-  (segment (start 81.28 152.4) (end 82.55 151.13) (width 0.95) (layer F.Cu) (net 72))
-  (segment (start 82.55 151.13) (end 82.55 147.32) (width 0.95) (layer F.Cu) (net 72))
-  (segment (start 82.55 147.32) (end 81.28 146.05) (width 0.95) (layer F.Cu) (net 72))
-  (segment (start 78.74 152.4) (end 81.28 152.4) (width 0.95) (layer F.Cu) (net 72))
-  (segment (start 109.22 152.4) (end 109.22 144.83) (width 0.95) (layer B.Cu) (net 82))
-  (segment (start 109.22 144.83) (end 109.4 144.65) (width 0.95) (layer B.Cu) (net 82))
-  (segment (start 103.4 130.45) (end 105.05 130.45) (width 0.95) (layer F.Cu) (net 83))
-  (segment (start 104.14 152.4) (end 106.68 152.4) (width 0.95) (layer F.Cu) (net 83))
-  (segment (start 101.6 149.86) (end 104.14 152.4) (width 0.95) (layer F.Cu) (net 83))
-  (segment (start 101.6 148.59) (end 101.6 149.86) (width 0.95) (layer F.Cu) (net 83))
-  (segment (start 104.14 146.05) (end 101.6 148.59) (width 0.95) (layer F.Cu) (net 83))
-  (segment (start 106.68 143.51) (end 104.14 146.05) (width 0.95) (layer F.Cu) (net 83))
-  (segment (start 106.68 132.08) (end 106.68 143.51) (width 0.95) (layer F.Cu) (net 83))
-  (segment (start 105.05 130.45) (end 106.68 132.08) (width 0.95) (layer F.Cu) (net 83))
-  (segment (start 113.03 132.82) (end 115.4 130.45) (width 0.95) (layer F.Cu) (net 84))
-  (segment (start 113.03 144.78) (end 113.03 132.82) (width 0.95) (layer F.Cu) (net 84))
-  (segment (start 115.57 147.32) (end 113.03 144.78) (width 0.95) (layer F.Cu) (net 84))
-  (segment (start 115.57 149.86) (end 115.57 147.32) (width 0.95) (layer F.Cu) (net 84))
-  (segment (start 113.03 152.4) (end 115.57 149.86) (width 0.95) (layer F.Cu) (net 84))
-  (segment (start 111.76 152.4) (end 113.03 152.4) (width 0.95) (layer F.Cu) (net 84))
-  (segment (start 113.03 148.59) (end 115.57 146.05) (width 0.95) (layer B.Cu) (net 168))
-  (segment (start 115.57 146.05) (end 115.57 142.82) (width 0.95) (layer B.Cu) (net 168))
-  (segment (start 115.57 142.82) (end 115.4 142.65) (width 0.95) (layer B.Cu) (net 168))
 )
